File: KiCad Project/TempControl4ch/TempControl4ch.kicad_pcb (KiCad board)
At the start: 2 copper layers, 100 x 60 mm, 76 parts, among them J1 Conn_01x08_Socket, J2 Conn_01x02_Socket, U1 MAX31856, U2 MAX31856, U3 MAX31856, U4 MAX31856, U5 BluePill_Part_Like_SWD_Breako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, U6 TPS54202DDC

Commit message: update pcb design
Other:
- board text added: "Mecha Dynamic - 4 ch Temperature Control Merve & Kaan ALKILINC"
Changed lines of the file:
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@@
 		(layer "Edge.Cuts")
 	)
+	(gr_text "Mecha Dynamic - 4 ch Temperature Control\nMerve & Kaan ALKILINC"
+		(at 118.2 61.6 90)
+		(layer "B.Cu")
+		(effects
+			(font
+				(size 1.5 1.5)
+				(thickness 0.3)
+				(bold yes)
+			)
+			(justify left bottom mirror)
+		)
+	)
 	(segment
 		(start 126.8 88)
@@
 		(start 169.75 80.6875)
 		(end 169.75 81.5)
-		(width 0.2)
+		(width 0.5)
 		(layer "F.Cu")
 		(net 2)
@@
 		(start 167.77 78.1225)
 		(end 167.77 80.6875)
-		(width 0.2)
+		(width 0.5)
 		(layer "F.Cu")
 		(net 2)
@@
 		(start 167.77 80.6875)
 		(end 169.75 80.6875)
-		(width 0.2)
+		(width 0.5)
 		(layer "F.Cu")
 		(net 2)
@@
 		(start 166 82.0425)
 		(end 167.77 83.8125)
-		(width 0.2)
+		(width 0.5)
 		(layer "F.Cu")
 		(net 6)
@@
 		(start 166 74)
 		(end 166.9975 74.9975)
-		(width 0.2)
+		(width 0.5)
 		(layer "F.Cu")
 		(net 6)
@@
 		(start 160.555 83.8125)
 		(end 167.77 83.8125)
-		(width 0.2)
+		(width 0.5)
 		(layer "F.Cu")
 		(net 6)
@@
 		(start 173.52 69.3225)
 		(end 170.625 69.3225)
-		(width 0.2)
+		(width 0.5)
 		(layer "F.Cu")
 		(net 6)
@@
 		(start 175.3875 78.505)
 		(end 175.3875 84.23)
-		(width 0.2)
+		(width 0.5)
 		(layer "F.Cu")
 		(net 6)
@@
 		(start 169.1875 83.8125)
 		(end 167.77 83.8125)
-		(width 0.2)
+		(width 0.5)
 		(layer "F.Cu")
 		(net 6)
@@
 		(start 169.75 82.5)
 		(end 169.75 83.25)
-		(width 0.2)
+		(width 0.5)
 		(layer "F.Cu")
 		(net 6)
@@
 		(start 170.625 69.3225)
 		(end 168.9475 71)
-		(width 0.2)
+		(width 0.5)
 		(layer "F.Cu")
 		(net 6)
@@
 		(start 168.9475 71)
 		(end 166 71)
-		(width 0.2)
+		(width 0.5)
 		(layer "F.Cu")
 		(net 6)
@@
 		(start 160.1375 84.23)
 		(end 160.555 83.8125)
-		(width 0.2)
+		(width 0.5)
 		(layer "F.Cu")
 		(net 6)
@@
 		(start 169.75 83.25)
 		(end 169.1875 83.8125)
-		(width 0.2)
+		(width 0.5)
 		(layer "F.Cu")
 		(net 6)
@@
 		(start 166 74)
 		(end 166 82.0425)
-		(width 0.2)
+		(width 0.5)
 		(layer "F.Cu")
 		(net 6)
@@
 		(start 166 71)
 		(end 166 74)
-		(width 0.2)
+		(width 0.5)
 		(layer "F.Cu")
 		(net 6)
@@
 		(start 139.01 62.8)
 		(end 133.48 68.33)
-		(width 0.2)
+		(width 0.5)
 		(layer "F.Cu")
 		(net 12)
@@
 		(start 133.48 68.33)
 		(end 133.48 69.305)
-		(width 0.2)
+		(width 0.5)
 		(layer "F.Cu")
 		(net 12)
@@
 		(start 128.485 62.8)
 		(end 121.98 69.305)
-		(width 0.2)
+		(width 0.5)
 		(layer "F.Cu")
 		(net 13)
@@
 		(start 135.2 62.8)
 		(end 128.485 62.8)
-		(width 0.2)
+		(width 0.5)
 		(layer "F.Cu")
 		(net 13)
@@
 		(start 167.75 72.405)
 		(end 170.5825 72.405)
-		(width 0.2)
+		(width 0.5)
 		(layer "F.Cu")
 		(net 16)
@@
 		(start 170.625 72.4475)
 		(end 170.625 74.9975)
-		(width 0.2)
+		(width 0.5)
 		(layer "F.Cu")
 		(net 16)
@@
 		(start 176.395 72.405)
 		(end 173.5625 72.405)
-		(width 0.2)
+		(width 0.5)
 		(layer "F.Cu")
 		(net 17)
@@
 		(start 173.52 72.4475)
 		(end 173.52 75.2275)
-		(width 0.2)
+		(width 0.5)
 		(layer "F.Cu")
 		(net 17)
@@
 		(start 142.82 62.8)
 		(end 137.23 68.39)
-		(width 0.2)
+		(width 0.5)
 		(layer "F.Cu")
 		(net 18)
@@
 		(start 137.23 68.39)
 		(end 137.23 69.305)
-		(width 0.2)
+		(width 0.5)
 		(layer "F.Cu")
 		(net 18)
@@
 		(start 150.44 62.8)
 		(end 150.44 67.245)
-		(width 0.2)
+		(width 0.5)
 		(layer "F.Cu")
 		(net 19)
@@
 		(start 150.44 67.245)
 		(end 152.5 69.305)
-		(width 0.2)
+		(width 0.5)
 		(layer "F.Cu")
 		(net 19)
@@
 		(start 154.64 62.8)
 		(end 161.145 69.305)
-		(width 0.2)
+		(width 0.5)
 		(layer "F.Cu")
 		(net 20)
@@
 		(start 154.25 62.8)
 		(end 154.64 62.8)
-		(width 0.2)
+		(width 0.5)
 		(layer "F.Cu")
 		(net 20)
@@
 		(start 169.89 62.8)
 		(end 176.395 69.305)
-		(width 0.2)
+		(width 0.5)
 		(layer "F.Cu")
 		(net 21)
@@
 		(start 161.87 62.8)
 		(end 169.89 62.8)
-		(width 0.2)
+		(width 0.5)
 		(layer "F.Cu")
 		(net 21)
@@
 		(start 176.395 69.305)
 		(end 179.25 69.305)
-		(width 0.2)
+		(width 0.5)
 		(layer "F.Cu")
 		(net 21)
@@
 		(start 162.396 67.136)
 		(end 165.581 67.136)
-		(width 0.2)
+		(width 0.5)
 		(layer "F.Cu")
 		(net 22)
@@
 		(start 158.06 62.8)
 		(end 162.396 67.136)
-		(width 0.2)
+		(width 0.5)
 		(layer "F.Cu")
 		(net 22)
@@
 		(start 165.581 67.136)
 		(end 167.75 69.305)
-		(width 0.2)
+		(width 0.5)
 		(layer "F.Cu")
 		(net 22)
@@
 		(start 146.63 68.565)
 		(end 145.89 69.305)
-		(width 0.2)
+		(width 0.5)
 		(layer "F.Cu")
 		(net 38)
@@
 		(start 146.63 62.8)
 		(end 146.63 68.565)
-		(width 0.2)
+		(width 0.5)
 		(layer "F.Cu")
 		(net 38)
@@
 		(start 172.17 107.75)
 		(end 183.5 107.75)
-		(width 0.4)
+		(width 0.5)
 		(layer "F.Cu")
 		(net 89)
@@
 		(start 165.93 113.99)
 		(end 172.17 107.75)
-		(width 0.4)
+		(width 0.5)
 		(layer "F.Cu")
 		(net 89)
@@
 			(pts
 				(xy 187.75 88.5) (xy 187.75 105.25) (xy 191.5 105.25) (xy 191.5 108) (xy 181.75 108) (xy 181.75 94.75)
-				(xy 185.75 88.5)
+				(xy 185 88.5)
 			)
 		)
